Commit message: Kinematics: base height 0.13 -> 0.17 (measured) in chain + URDF
EE at home now (0,0,0.837). Shifts the whole arm +4cm in absolute Z (waist is a
yaw joint, so relative kinematics unchanged). Deployed to the Pi.

File: urdf/moveo.urdf (robot description, URDF)
Before this commit: robot moveo, 7 links, 6 joints
Links:
- link base_link: geometry visual cylinder length=0.170 radius=0.045
Joints:
- joint Joint_1: origin xyz=0 0 0.130 rpy=0 0 0 -> xyz=0 0 0.170 rpy=0 0 0

Commit message: Fix ESP USB transport, IK frame/seeding, j4 dir; add camera mount
Firmware:
- Reverse j4 (wrist roll) direction (DIR_INVERT[3]=false) per measured behaviour.

ESP flashing (root-caused a total micro-ROS comms loss):
- flash_esp32_from_pi.sh: FQBN was missing :CDCOnBoot=cdc, which routed Serial
  (the micro-ROS transport) to UART0 pins instead of USB -> agent saw silence.
  Also fixed stale agent baud (115200) and port (/dev/ttyACM0).
- flash_esp32_usb.sh: new flash via esptool USB self-reset (no GPIO), avoids the
  gpioset bootloader hang; logs to ~/flash2.log (survives /tmp cleaning).
- esp_diag.py / reconnect_esp.sh: ESP boot-capture + agent recovery helpers.

IK (moveo_publisher.py):
- Fix +X targets resolving to a contorted 'reach-behind' pose (and -X crashing):
  the home seed is a waist singularity; aim the seed at the target azimuth and add
  a naturalness tiebreaker (penalise 180-deg wrist roll). Harden the no-solution path.
- Rotate the base frame to REP-103 (+X forward, +Y left): user commands are now
  rotated -90 deg about Z into the internal chain frame inside solve_ik.

URDF:
- Add eye-in-hand stereo camera mount (camera_mount + left/right) from the CAD:
  midpoint -0.05 X, cameras +/-0.03 Y in the EE frame, optical axis +Z.

Vision:
- start_vision.sh: camera remounted right-way-up -> drop the cosmetic 180 display
  rotation so the stream is upright. (Stereo depth still needs recal for new mount.)

run_moveo_publisher.sh: detached publisher restart with a proper bind wait.

File: urdf/moveo.urdf (robot description, URDF)
Before this commit: robot moveo, 7 links, 6 joints
Links:
- added link camera_mount; visual box size=0.018 0.080 0.018
- added link left_camera; visual box size=0.015 0.015 0.015
- added link right_camera; visual box size=0.015 0.015 0.015
Joints:
- added joint camera_mount_joint: type fixed, parent ee_link, child camera_mount, origin xyz=-0.05 0 0 rpy=0 0 0
- added joint left_camera_joint: type fixed, parent camera_mount, child left_camera, origin xyz=0 -0.03 0 rpy=0 0 0
- added joint right_camera_joint: type fixed, parent camera_mount, child right_camera, origin xyz=0 0.03 0 rpy=0 0 0

Commit message: feat(kinematics): unify FK/IK with single source of truth in kinematics.py + corrected lengths (BASE=0.20, WAIST=0.140, UPPER=0.22, FORE=0.11, WRIST=0.11, EE=0.06)
- Make software/mac-gui/kinematics.py the canonical definition (lengths + Chain).
- Update both moveo_publisher.py (Mac + Pi) to use it (import on Mac, try-import + fallback on Pi).
- Fix user-frame convention: forward_kinematics now returns +X forward / +Y left so Compute FK button matches IK targets.
- Correct 2R pre-solve for non-zero WAIST.
- Pi TCP response now includes 'achieved' (user-frame) for immediate verification in logs.
- Higher angle precision on wire + safer restart in deploy.
- Deployed updated files to Pi; FK/IK now match.

Addresses long-standing FK/IK mismatch (e.g. target 0.25/0/0.3 now recovers correctly from joints).

File: urdf/moveo.urdf (robot description, URDF)
Before this commit: robot moveo, 10 links, 9 joints
Links:
- removed link camera_mount
- removed link ee_link
- removed link left_camera
- removed link right_camera
- link Link_1: mass 0.8 -> 4.2526; geometry collision mesh filename=package://moveo_description/meshes/Link_1_col.stl; visual mesh filename=package://moveo_description/meshes/Link_1.stl
- link Link_2: mass 0.6 -> 1.9323; geometry collision mesh filename=package://moveo_description/meshes/Link_2_col.stl; visual mesh filename=package://moveo_description/meshes/Link_2.stl
- link Link_3: mass 0.4 -> 1.1381; geometry collision mesh filename=package://moveo_description/meshes/Link_3_col.stl; visual mesh filename=package://moveo_description/meshes/Link_3.stl
- link Link_4: mass 0.2 -> 0.62964; geometry collision mesh filename=package://moveo_description/meshes/Link_4_col.stl; visual mesh filename=package://moveo_description/meshes/Link_4.stl
- link Link_5: mass 0.15 -> 0.19875; geometry collision mesh filename=package://moveo_description/meshes/Link_5_col.stl; visual mesh filename=package://moveo_description/meshes/Link_5.stl
- link base_link: mass 1.0 -> None; geometry collision mesh filename=package://moveo_description/meshes/base_link_col.stl; visual mesh filename=package://moveo_description/meshes/base_link.stl
Joints:
- removed joint Joint_ee
- removed joint camera_mount_joint
- removed joint left_camera_joint
- removed joint right_camera_joint
- joint Joint_1: axis 0 0 1 -> 0 1 0; limit lower=-2.00 upper=2.40 effort=10 velocity=2 -> lower=-1.5707 upper=1.5707 effort=5 velocity=1; origin xyz=0 0 0.170 rpy=0 0 0 -> xyz=0.00000000 -0.24250000 0.13000000 rpy=1.57079633 0.00000367 1.20579347
- joint Joint_2: axis 1 0 0 -> 0 -1 0; limit lower=-1.95 upper=1.95 effort=10 velocity=2 -> lower=-1.5707 upper=1.5707 effort=5 velocity=1; origin xyz=0 0 0.183 rpy=0 0 0 -> xyz=0.00000000 0.18264000 0.00000000 rpy=1.57078667 1.57079206 0.00000000
- joint Joint_3: axis 1 0 0 -> 0 -1 0; limit lower=-2.20 upper=2.20 effort=10 velocity=2 -> lower=-1.5707 upper=1.5707 effort=5 velocity=1; origin xyz=0 0 0.221 rpy=0 0 0 -> xyz=0.00000000 0.00000000 -0.22112000 rpy=0.00000124 1.56835920 0.00000000
- joint Joint_4: axis 0 0 1 -> 0.010353 -0.99993 -0.0059382; limit lower=-3.14 upper=3.14 effort=10 velocity=2 -> lower=-1.5707 upper=1.5707 effort=5 velocity=1; origin xyz=0 0 0.170 rpy=0 0 0 -> xyz=0.16988000 -0.00099213 0.00000000 rpy=-0.04402676 1.00297628 -1.60635499
- joint Joint_5: axis 1 0 0 -> 0 1 0; limit lower=-1.75 upper=1.75 effort=10 velocity=2 -> lower=-1.5707 upper=1.5707 effort=5 velocity=1; origin xyz=0 0 0.053 rpy=0 0 0 -> xyz=-0.00213460 0.05304100 0.00169360 rpy=-1.48048705 0.01406373 -1.64986156
